Commit message: feat: add distinct sensor visual palette

File: ros1_ws/src/wildebeest_description/urdf/materials.xacro (robot description, xacro)
@@ -10,6 +10,20 @@
     <color rgba="0.1 0.82 0.68 1.0"/>
   </material>
-  <material name="sensor_black">
-    <color rgba="0.015 0.02 0.025 1.0"/>
+  <!-- High-contrast sensor identification palette. These colors identify
+       hardware in RViz/Gazebo; they do not report sensor health or status. -->
+  <material name="sensor_lidar_orange">
+    <color rgba="0.902 0.624 0.000 1.0"/>
+  </material>
+  <material name="sensor_imu_rose">
+    <color rgba="0.800 0.475 0.655 1.0"/>
+  </material>
+  <material name="sensor_gnss_yellow">
+    <color rgba="0.941 0.894 0.259 1.0"/>
+  </material>
+  <material name="sensor_camera_sky_blue">
+    <color rgba="0.337 0.706 0.914 1.0"/>
+  </material>
+  <material name="sensor_ultrasonic_vermillion">
+    <color rgba="0.835 0.369 0.000 1.0"/>
   </material>
 </robot>

File: ros1_ws/src/wildebeest_description/urdf/wildebeest.gazebo.xacro (robot description, xacro)
@@ -23,4 +23,5 @@
     </gazebo>
     <gazebo reference="${prefix}lidar_link">
+      <material>Wildebeest/SensorLidarOrange</material>
       <sensor name="lidar" type="ray">
         <always_on>true</always_on><update_rate>10</update_rate><visualize>true</visualize>
@@ -37,4 +38,5 @@
     </gazebo>
     <gazebo reference="${prefix}camera_link">
+      <material>Wildebeest/SensorCameraSkyBlue</material>
       <sensor name="front_camera" type="camera">
         <always_on>true</always_on><update_rate>20</update_rate><visualize>false</visualize>
@@ -51,4 +53,5 @@
     </gazebo>
     <gazebo reference="${prefix}imu_link">
+      <material>Wildebeest/SensorImuRose</material>
       <sensor name="imu" type="imu">
         <always_on>true</always_on><update_rate>50</update_rate>
@@ -60,4 +63,5 @@
     </gazebo>
     <gazebo reference="${prefix}ultrasonic_front_link">
+      <material>Wildebeest/SensorUltrasonicVermillion</material>
       <sensor name="front_ultrasonic" type="ray">
         <always_on>true</always_on><update_rate>10</update_rate>
@@ -71,4 +75,7 @@
         </plugin>
       </sensor>
+    </gazebo>
+    <gazebo reference="${prefix}gps_link">
+      <material>Wildebeest/SensorGnssYellow</material>
     </gazebo>
     <xacro:if value="${simulate_gps}">

File: ros1_ws/src/wildebeest_description/urdf/wildebeest.urdf.xacro (robot description, xacro)
@@ -112,5 +112,5 @@
     <visual>
       <geometry><cylinder radius="0.047" length="0.055"/></geometry>
-      <material name="sensor_black"/>
+      <material name="sensor_lidar_orange"/>
     </visual>
     <collision><geometry><cylinder radius="0.047" length="0.055"/></geometry></collision>
@@ -122,5 +122,5 @@
   </joint>
   <link name="${prefix}imu_link">
-    <visual><geometry><box size="0.026 0.020 0.006"/></geometry><material name="wildebeest_accent"/></visual>
+    <visual><geometry><box size="0.026 0.020 0.006"/></geometry><material name="sensor_imu_rose"/></visual>
     <inertial><mass value="0.01"/><inertia ixx="0.000001" ixy="0" ixz="0" iyy="0.000001" iyz="0" izz="0.000001"/></inertial>
   </link>
@@ -130,5 +130,5 @@
   </joint>
   <link name="${prefix}gps_link">
-    <visual><geometry><box size="0.045 0.045 0.010"/></geometry><material name="wildebeest_accent"/></visual>
+    <visual><geometry><box size="0.045 0.045 0.010"/></geometry><material name="sensor_gnss_yellow"/></visual>
     <xacro:box_inertial mass="0.02" x="0.045" y="0.045" z="0.010"/>
   </link>
@@ -138,5 +138,5 @@
   </joint>
   <link name="${prefix}camera_link">
-    <visual><geometry><box size="0.025 0.050 0.025"/></geometry><material name="sensor_black"/></visual>
+    <visual><geometry><box size="0.025 0.050 0.025"/></geometry><material name="sensor_camera_sky_blue"/></visual>
     <collision><geometry><box size="0.025 0.050 0.025"/></geometry></collision>
     <xacro:box_inertial mass="0.035" x="0.025" y="0.050" z="0.025"/>
@@ -152,5 +152,5 @@
   </joint>
   <link name="${prefix}ultrasonic_front_link">
-    <visual><origin rpy="0 ${pi/2.0} 0"/><geometry><cylinder radius="0.019" length="0.015"/></geometry><material name="sensor_black"/></visual>
+    <visual><origin rpy="0 ${pi/2.0} 0"/><geometry><cylinder radius="0.019" length="0.015"/></geometry><material name="sensor_ultrasonic_vermillion"/></visual>
     <xacro:box_inertial mass="0.01" x="0.015" y="0.038" z="0.038"/>
   </link>

File: ros2_ws/src/wildebeest_description/urdf/materials.xacro (robot description, xacro)
@@ -13,12 +13,23 @@
     <color rgba="0.018 0.022 0.028 1.0"/>
   </material>
-  <material name="wildebeest_silver">
-    <color rgba="0.55 0.60 0.65 1.0"/>
-  </material>
   <material name="wildebeest_green">
     <color rgba="0.10 0.62 0.30 1.0"/>
   </material>
-  <material name="wildebeest_red">
-    <color rgba="0.82 0.08 0.10 1.0"/>
+  <!-- Sensor-only colors are based on the color-blind-conscious Okabe-Ito
+       palette.  Their semantic names keep RViz and Gazebo visuals legible. -->
+  <material name="wildebeest_sensor_lidar_orange">
+    <color rgba="0.902 0.624 0.000 1.0"/>
+  </material>
+  <material name="wildebeest_sensor_imu_rose">
+    <color rgba="0.800 0.475 0.655 1.0"/>
+  </material>
+  <material name="wildebeest_sensor_gnss_yellow">
+    <color rgba="0.941 0.894 0.259 1.0"/>
+  </material>
+  <material name="wildebeest_sensor_camera_sky">
+    <color rgba="0.337 0.706 0.914 1.0"/>
+  </material>
+  <material name="wildebeest_sensor_ultrasonic_vermillion">
+    <color rgba="0.835 0.369 0.000 1.0"/>
   </material>
 </robot>

File: ros2_ws/src/wildebeest_description/urdf/wildebeest.urdf.xacro (robot description, xacro)
@@ -96,5 +96,5 @@
     <visual>
       <geometry><cylinder radius="0.047" length="0.055"/></geometry>
-      <material name="wildebeest_graphite"/>
+      <material name="wildebeest_sensor_lidar_orange"/>
     </visual>
     <collision><geometry><cylinder radius="0.047" length="0.055"/></geometry></collision>
@@ -109,5 +109,5 @@
     <visual>
       <geometry><box size="0.022 0.017 0.004"/></geometry>
-      <material name="wildebeest_red"/>
+      <material name="wildebeest_sensor_imu_rose"/>
     </visual>
     <xacro:box_inertial mass="0.003" x="0.022" y="0.017" z="0.004"/>
@@ -121,5 +121,5 @@
     <visual>
       <geometry><box size="0.035 0.025 0.008"/></geometry>
-      <material name="wildebeest_green"/>
+      <material name="wildebeest_sensor_gnss_yellow"/>
     </visual>
     <xacro:box_inertial mass="0.012" x="0.035" y="0.025" z="0.008"/>
@@ -133,5 +133,5 @@
     <visual>
       <geometry><box size="0.025 0.032 0.032"/></geometry>
-      <material name="wildebeest_graphite"/>
+      <material name="wildebeest_sensor_camera_sky"/>
     </visual>
     <collision><geometry><box size="0.025 0.032 0.032"/></geometry></collision>
@@ -153,5 +153,5 @@
       <origin rpy="0 ${pi / 2.0} 0"/>
       <geometry><cylinder radius="0.019" length="0.015"/></geometry>
-      <material name="wildebeest_silver"/>
+      <material name="wildebeest_sensor_ultrasonic_vermillion"/>
     </visual>
     <xacro:cylinder_inertial mass="0.009" radius="0.019" length="0.015" origin_rpy="0 ${pi / 2.0} 0"/>
